Commit message: Fixed Joints
Saw post about joints not supposed to disconnect, initially thought was just errant behavior of engine, fixed it to be fixed in position

File: body.urdf (robot description, URDF)
Before this commit: robot robot, 3 links, 2 joints
Joints:
- joint Torso_Leg_Back: origin xyz=rx-0.5 ry rz-0.5 rpy=0 0 0 -> xyz=-0.5 0 1 rpy=0 0 0
- joint Torso_Leg_Front: origin xyz=rx+0.5 ry rz-0.5 rpy=0 0 0 -> xyz=0.5 0 1 rpy=0 0 0

Commit message: Finished Neurons
Forgot to commit when initially finished

File: body.urdf (robot description, URDF)
Before this commit: robot robot, 3 links, 2 joints
Links:
- removed link Back_Leg
- removed link Front_Leg
- added link BackLeg, mass 1; collision box size=1 1 1; visual box size=1 1 1
- added link FrontLeg, mass 1; collision box size=1 1 1; visual box size=1 1 1
Joints:
- removed joint Torso_Leg_Back
- removed joint Torso_Leg_Front
- added joint Torso_BackLeg: type revolute, parent Torso, child BackLeg, origin xyz=1 0 1 rpy=0 0 0, axis 0 1 0, limit lower=-3.14159 upper=3.14159 effort=0.0 velocity=0.0
- added joint Torso_FrontLeg: type revolute, parent Torso, child FrontLeg, origin xyz=2 0 1 rpy=0 0 0, axis 0 1 0, limit lower=-3.14159 upper=3.14159 effort=0.0 velocity=0.0
